Commit message: testing

File: visual_servoing/apple_ws/src/robot_servoing/model/urdf/demo_apple.urdf.xacro (robot description, xacro)
@@ -72,23 +72,23 @@
   </link>
   <link name="apple_link">
-  <visual>
-    <origin xyz="0 0 0" rpy="0 0 0"/>
-    <geometry>
-      <sphere radius="${apple_radius}"/>
-    </geometry>
-    <material name="red"/>
-  </visual>
-  <collision>
-    <origin xyz="0 0 0" rpy="0 0 0"/>
-    <geometry>
-      <sphere radius="${apple_radius}"/>
-    </geometry>
-  </collision>
-  <inertial>
-    <mass value="${apple_mass}"/>
-    <origin xyz="0 0 0"/>
-    <inertia ixx="0.0001" iyy="0.0001" izz="0.0001" ixy="0" ixz="0" iyz="0"/>
-  </inertial>
-</link>
+    <visual>
+      <origin xyz="0 0 0" rpy="0 0 ${pi/2}"/>
+      <geometry>
+        <box size="0.05 0.15 0.15" />
+      </geometry>
+      <material name="black"/>
+    </visual>
+    <collision>
+      <origin xyz="0 0 0" rpy="0 0 0"/>
+      <geometry>
+        <box size="0.1 0.15 0.15" />
+      </geometry>
+    </collision>
+    <inertial>
+      <mass value="${apple_mass}"/>
+      <origin xyz="0 0 0"/>
+      <inertia ixx="0.0001" iyy="0.0001" izz="0.0001" ixy="0" ixz="0" iyz="0"/>
+    </inertial>
+  </link>
   <joint name="pole_base_joint" type="fixed">
     <parent link="world"/>

File: visual_servoing/apple_ws/src/robot_servoing/model/urdf/robot.urdf.xacro (robot description, xacro)
@@ -5,4 +5,4 @@
   <xacro:include filename="$(find robot_servoing)/model/urdf/sim_interface.urdf.xacro" />
   <xacro:include filename="$(find robot_servoing)/model/urdf/ur_camera.urdf.xacro" />
-  <xacro:include filename="$(find robot_servoing)/model/urdf/demo_apple.urdf.xacro" />
+  <!-- <xacro:include filename="$(find robot_servoing)/model/urdf/demo_apple.urdf.xacro" /> -->
 </robot>

File: visual_servoing/apple_ws/src/robot_servoing/model/urdf/ur_camera.urdf.xacro (robot description, xacro)
@@ -62,5 +62,5 @@
      name="$(arg name)"
      tf_prefix="$(arg tf_prefix)"
-     parent="world"
+     parent="slider_link"
      joint_limits_parameters_file="$(arg joint_limit_params)"
      kinematics_parameters_file="$(arg kinematics_params)"
@@ -96,5 +96,5 @@
      trajectory_port="$(arg trajectory_port)"
      >
-     <origin xyz="0 0 0" rpy="0 0 0" />          <!-- position robot in the world -->
+     <origin xyz="0 0 0.03" rpy="0 0 0" />          <!-- position robot in the world -->
    </xacro:ur_robot>
    <xacro:if value="$(arg sim_gazebo)">
@@ -119,4 +119,44 @@
     </gazebo>
   </xacro:if>
+  <!-- Box -->
+  <link name="box_link">
+    <visual>
+      <origin xyz="0 0 0" rpy="0 0 0"/>
+      <geometry>
+        <box size="2 0.5 0.5" />
+      </geometry>
+      <material name="black"/>
+    </visual>
+    <collision>
+      <origin xyz="0 0 0" rpy="0 0 0"/>
+      <geometry>
+        <box size="0.5 0.5 0.5" />
+      </geometry>
+    </collision>
+    <inertial>
+      <mass value="5.0"/>
+      <origin xyz="0 0 0"/>
+      <inertia ixx="0.1" iyy="0.1" izz="0.1" ixy="0" ixz="0" iyz="0"/>
+    </inertial>
+  </link>
+    <link name="slider_link">
+    <visual>
+      <origin xyz="0 0 0" rpy="0 0 0"/>
+      <geometry>
+        <box size="0.25 0.25 0.05" />
+      </geometry>
+      <material name="white"/>
+    </visual>
+    <collision>
+      <origin xyz="0 0 0" rpy="0 0 0"/>
+      <geometry>
+        <box size="0.25 0.25 0.05" />
+      </geometry>
+    </collision>
+    <inertial>
+      <mass value="1000"/>
+      <inertia ixx="4.4" ixy="0.0" ixz="0.0" iyy="4.4" iyz="0.0" izz="0.2"/>
+    </inertial>
+  </link>
   <!-- Camera body -->
   <link name="camera_body_link">
@@ -159,4 +199,10 @@
   <!-- Camera sensor link -->
   <link name="camera_link"/>
+  <link name="camera_link_sensor"/>
+  <joint name="camera_sensor_joint_frame" type="fixed">
+    <origin xyz="0 0 0" rpy="-${pi/2} 0 -${pi/2}"/>
+    <parent link="camera_link"/>
+    <child link="camera_link_sensor"/>
+  </joint>
   <!-- joints -->
   <joint name="camera_sensor_joint" type="fixed">
@@ -175,3 +221,29 @@
     <origin xyz="0 0 0.015" rpy="${pi/2} -${pi/2} 0" />
   </joint>
+  <joint name="box_to_world_joint" type="fixed">
+    <origin xyz="0 0 0.25" rpy="0 0 0"/>
+    <parent link="world"/>
+    <child link="box_link"/>
+  </joint>
+  <joint name="slider_joint" type="prismatic">
+    <origin xyz="0 0 0.3" rpy="0 0 0"/>
+    <parent link="box_link"/>
+    <child link="slider_link"/>
+    <axis xyz="1 0 0"/> <!-- Axis of sliding -->
+    <limit effort="0.0" lower="-1.0" upper="1.0" velocity="1.0"/>
+  </joint>
+  <ros2_control name="ur_slider_control" type="system">
+    <hardware>
+      <plugin>ign_ros2_control/IgnitionSystem</plugin>
+    </hardware>
+    <joint name="slider_joint">
+       <command_interface name="position"/>
+       <command_interface name="velocity"/>
+       <state_interface name="position">
+         <!-- initial position for the FakeSystem and simulation -->
+         <param name="initial_value">0.0</param>
+       </state_interface>
+       <state_interface name="velocity"/>
+    </joint>
+  </ros2_control>
 </robot>
